Commit message: Fixed even more file path issues, added 3D model to gazebo environment.

File: src/hw_gazebo/urdf/mogi_bot.urdf (robot description, URDF)
Before this commit: robot mogi_bot, 8 links, 7 joints
Links:
- link base_link: geometry collision box size=.4 .2 .1; collision sphere radius=0.0499
- link left_wheel: geometry collision cylinder length=.05 radius=.1; visual mesh filename=package://hw_gazebo/meshes/wheel.dae
- link right_wheel: geometry collision cylinder length=.05 radius=.1; visual mesh filename=package://hw_gazebo/meshes/wheel.dae

Commit message: Replaced robot with 4 wheeler

File: src/hw_gazebo/urdf/mogi_bot.urdf (robot description, URDF)
Before this commit: robot mogi_bot, 8 links, 7 joints
Links:
- removed link camera_link
- removed link camera_link_optical
- removed link left_wheel
- removed link right_wheel
- added link front_left_wheel, mass 2.0; collision sphere radius=.1; visual mesh filename=package://hw_gazebo/meshes/mecanum_wheel_left.STL scale=0.002 .002 0.002
- added link front_right_wheel, mass 2.0; collision sphere radius=.1; visual mesh filename=package://hw_gazebo/meshes/mecanum_wheel_right.STL scale=0.002 .002 0.002
- added link rear_left_wheel, mass 2.0; collision sphere radius=.1; visual mesh filename=package://hw_gazebo/meshes/mecanum_wheel_right.STL scale=0.002 .002 0.002
- added link rear_right_wheel, mass 2.0; collision sphere radius=.1; visual mesh filename=package://hw_gazebo/meshes/mecanum_wheel_left.STL scale=0.002 .002 0.002
- link base_link: geometry collision box size=.4 .2 .1; visual mesh filename=package://hw_gazebo/meshes/mogi_bot.dae
Joints:
- removed joint camera_joint
- removed joint camera_optical_joint
- removed joint left_wheel_joint
- removed joint right_wheel_joint
- added joint front_left_wheel_joint: type continuous, parent base_link, child front_left_wheel, origin xyz=0.15 0.15 0 rpy=-1.5707 0 0, axis 0 0 1, limit effort=10000 velocity=10
- added joint front_right_wheel_joint: type continuous, parent base_link, child front_right_wheel, origin xyz=0.15 -0.15 0 rpy=-1.5707 0 0, axis 0 0 1, limit effort=10000 velocity=10
- added joint rear_left_wheel_joint: type continuous, parent base_link, child rear_left_wheel, origin xyz=-0.15 0.15 0 rpy=-1.5707 0 0, axis 0 0 1, limit effort=10000 velocity=10
- added joint rear_right_wheel_joint: type continuous, parent base_link, child rear_right_wheel, origin xyz=-0.15 -0.15 0 rpy=-1.5707 0 0, axis 0 0 1, limit effort=10000 velocity=10
